Commit message: update: moveit2 package fixed for stretch arm

File: stretch_moveit_config/config/stretch.ros2_control.xacro (robot description, xacro)
@@ -64,5 +64,19 @@
                 <state_interface name="velocity"/>
             </joint>
-            <!-- <joint name="joint_gripper_finger_left">
+            <joint name="joint_head_pan">
+                <command_interface name="position"/>
+                <state_interface name="position">
+                  <param name="initial_value">${initial_positions['joint_head_pan']}</param>
+                </state_interface>
+                <state_interface name="velocity"/>
+            </joint>
+            <joint name="joint_head_tilt">
+                <command_interface name="position"/>
+                <state_interface name="position">
+                  <param name="initial_value">${initial_positions['joint_head_tilt']}</param>
+                </state_interface>
+                <state_interface name="velocity"/>
+            </joint>
+            <joint name="joint_gripper_finger_left">
                 <command_interface name="position"/>
                 <state_interface name="position">
@@ -77,19 +91,5 @@
                 </state_interface>
                 <state_interface name="velocity"/>
-            </joint> -->
-            <!-- <joint name="joint_head_pan">
-                <command_interface name="position"/>
-                <state_interface name="position">
-                  <param name="initial_value">${initial_positions['joint_head_pan']}</param>
-                </state_interface>
-                <state_interface name="velocity"/>
             </joint>
-            <joint name="joint_head_tilt">
-                <command_interface name="position"/>
-                <state_interface name="position">
-                  <param name="initial_value">${initial_positions['joint_head_tilt']}</param>
-                </state_interface>
-                <state_interface name="velocity"/>
-            </joint> -->
         </ros2_control>
     </xacro:macro>
