Commit message: Update stretch setup and moveit2 for all joints

File: stretch_plugin_config/config/stretch.ros2_control.xacro (robot description, xacro)
@@ -8,4 +8,5 @@
                 <plugin>mock_components/GenericSystem</plugin>
             </hardware>
+            <!-- ARM JOINTS-->
             <joint name="joint_lift">
                 <command_interface name="position"/>
@@ -64,4 +65,5 @@
                 <state_interface name="velocity"/>
             </joint>
+            <!-- BASE JOINTS -->
             <joint name="joint_left_wheel">
                 <command_interface name="position"/>
@@ -78,4 +80,34 @@
                 <state_interface name="velocity"/>
             </joint>
+            <!-- HEAD JOINTS -->
+            <joint name="joint_head_pan">
+                <command_interface name="position"/>
+                <state_interface name="position">
+                  <param name="initial_value">${initial_positions['joint_head_pan']}</param>
+                </state_interface>
+                <state_interface name="velocity"/>
+            </joint>
+            <joint name="joint_head_tilt">
+                <command_interface name="position"/>
+                <state_interface name="position">
+                  <param name="initial_value">${initial_positions['joint_head_tilt']}</param>
+                </state_interface>
+                <state_interface name="velocity"/>
+            </joint>
+            <!-- GRIPPER JOINTS -->
+            <joint name="joint_gripper_finger_left">
+                <command_interface name="position"/>
+                <state_interface name="position">
+                  <param name="initial_value">${initial_positions['joint_gripper_finger_left']}</param>
+                </state_interface>
+                <state_interface name="velocity"/>
+            </joint>
+            <joint name="joint_gripper_finger_right">
+                <command_interface name="position"/>
+                <state_interface name="position">
+                  <param name="initial_value">${initial_positions['joint_gripper_finger_right']}</param>
+                </state_interface>
+                <state_interface name="velocity"/>
+            </joint>
         </ros2_control>
     </xacro:macro>
